Commit message: update the birngup launch file and add gmapping launch file

File: urdf/ARC_RCcar.urdf.xacro (robot description, xacro)
@@ -7,8 +7,8 @@
     <xacro:arg name="camera_name"   default="zed" />
     <xacro:arg name="camera_model"  default="zed" />
-    <xacro:arg name="base_frame"    default="zed_base_link" />
-    <xacro:arg name="cam_pos_x"     default="0.0" />
+    <xacro:arg name="base_frame"    default="base_link" />
+    <xacro:arg name="cam_pos_x"     default="0.40" />
     <xacro:arg name="cam_pos_y"     default="0.0" />
-    <xacro:arg name="cam_pos_z"     default="0.0" />
+    <xacro:arg name="cam_pos_z"     default="0.065" />
     <xacro:arg name="cam_roll"      default="0.0" />
     <xacro:arg name="cam_pitch"     default="0.0" />
@@ -107,11 +107,11 @@
   <xacro:macro name="right_wheels_collision_geometry">
     <origin xyz="0 0 0.0225" rpy="0 0 0" />
-    <geometry>e="robot_description"/>
+    <geometry>
       <cylinder length="0.045" radius="0.05" />
     </geometry>
   </xacro:macro>
   <!-- ADD chassis and its inertia link -->
-  <link name="$(arg robot_name)_base_link"/>
-  <link name="$(arg robot_name)_chassis">
+  <link name="base_link"/>
+  <link name="chassis">
     <visual>
       <xacro:chassis_geometry/>
@@ -119,21 +119,21 @@
     </visual>
   </link>
-  <joint name="$(arg robot_name)_base_link_joint" type="fixed">
+  <joint name="base_link_joint" type="fixed">
     <origin xyz="0 0 0.05" rpy="0 0 0" />
-    <parent link="$(arg robot_name)_base_link" />
-    <child link="$(arg robot_name)_chassis" />
-  </joint>
-  <link name="$(arg robot_name)_chassis_inertia">
+    <parent link="base_link" />
+    <child link="chassis" />
+  </joint>
+  <link name="chassis_inertia">
     <inertial>
       <xacro:chassis_inertial_params />
     </inertial>
   </link>
-  <joint name="$(arg robot_name)_chassis_inertia_joint" type="fixed">
-    <origin xyz="0 0 0" rpy="0 0 0" />
-    <parent link="$(arg robot_name)_chassis" />
-    <child link="$(arg robot_name)_chassis_inertia" />
+  <joint name="chassis_inertia_joint" type="fixed">
+    <origin xyz="0 0 0" rpy="0 0 0" />
+    <parent link="chassis" />
+    <child link="chassis_inertia" />
   </joint>
   <!-- Add the left rear wheel with its joints -->
-  <link name="$(arg robot_name)_left_rear_wheel">
+  <link name="left_rear_wheel">
     <inertial>
       <xacro:left_wheels_inertial_params />
@@ -147,13 +147,13 @@
     </collision>
   </link>
-  <joint name="$(arg robot_name)_left_rear_wheel_joint" type="continuous">
+  <joint name="left_rear_wheel_joint" type="continuous">
     <origin xyz="0 0.1 0" rpy="1.5708 0 0" />
-    <parent link="$(arg robot_name)_chassis" />
-    <child link="$(arg robot_name)_left_rear_wheel" />
+    <parent link="chassis" />
+    <child link="left_rear_wheel" />
     <axis xyz="0 0 -1" />
     <limit effort="10" velocity="100" />
   </joint>
     <!-- Add the right rear wheel with its joints -->
-  <link name="$(arg robot_name)_right_rear_wheel">
+  <link name="right_rear_wheel">
     <inertial>
       <xacro:right_wheels_inertial_params />
@@ -167,13 +167,13 @@
     </collision>
   </link>
-  <joint name="$(arg robot_name)_right_rear_wheel_joint" type="continuous">
+  <joint name="right_rear_wheel_joint" type="continuous">
     <origin xyz="0 -0.1 0" rpy="1.5708 0 0" />
-    <parent link="$(arg robot_name)_chassis" />
-    <child link="$(arg robot_name)_right_rear_wheel" />
+    <parent link="chassis" />
+    <child link="right_rear_wheel" />
     <axis xyz="0 0 -1" />
     <limit effort="10" velocity="100" />
   </joint>
  <!-- Add the steering hinge and its joints -->
- <link name="$(arg robot_name)_left_steering_hinge">
+ <link name="left_steering_hinge">
     <inertial>
       <xacro:steering_hinge_inertial_params />
@@ -184,12 +184,12 @@
     </visual>
   </link>
-  <joint name="$(arg robot_name)_left_steering_hinge_joint" type="revolute">
+  <joint name="left_steering_hinge_joint" type="revolute">
     <origin xyz="0.325 0.1 0" rpy="0 1.5708 0" />
-    <parent link="$(arg robot_name)_chassis" />
-    <child link="$(arg robot_name)_left_steering_hinge" />
+    <parent link="chassis" />
+    <child link="left_steering_hinge" />
     <axis xyz="-1 0 0" />
     <limit lower="-1.0" upper="1.0" effort="10" velocity="100" />
   </joint>
-  <link name="$(arg robot_name)_right_steering_hinge">
+  <link name="right_steering_hinge">
     <inertial>
       <xacro:steering_hinge_inertial_params />
@@ -200,13 +200,13 @@
     </visual>
   </link>
-  <joint name="$(arg robot_name)_right_steering_hinge_joint" type="continuous">
+  <joint name="right_steering_hinge_joint" type="continuous">
     <origin xyz="0.325 -0.1 0" rpy="0 1.5708 0" />
-    <parent link="$(arg robot_name)_chassis" />
-    <child link="$(arg robot_name)_right_steering_hinge" />
+    <parent link="chassis" />
+    <child link="right_steering_hinge" />
     <axis xyz="-1 0 0" />
     <limit lower="-1.0" upper="1.0" effort="10" velocity="100" />
   </joint>
 <!-- Add the left front wheel with its joints and tranmissions -->
-  <link name="$(arg robot_name)_left_front_wheel">
+  <link name="left_front_wheel">
     <inertial>
       <xacro:left_wheels_inertial_params />
@@ -220,13 +220,13 @@
     </collision>
   </link>
-  <joint name="$(arg robot_name)_left_front_wheel_joint" type="continuous">
+  <joint name="left_front_wheel_joint" type="continuous">
     <origin xyz="0 0 0" rpy="1.5708 0 0" />
-    <parent link="$(arg robot_name)_left_steering_hinge" />
-    <child link="$(arg robot_name)_left_front_wheel" />
+    <parent link="left_steering_hinge" />
+    <child link="left_front_wheel" />
     <axis xyz="0 0 -1" />
     <limit effort="10" velocity="100" />
   </joint>
     <!-- Add the right front wheel with its joints and tranmissions -->
-  <link name="$(arg robot_name)_right_front_wheel">
+  <link name="right_front_wheel">
     <inertial>
       <xacro:right_wheels_inertial_params />
@@ -240,13 +240,13 @@
     </collision>
   </link>
-  <joint name="$(arg robot_name)_right_front_wheel_joint" type="continuous">
+  <joint name="right_front_wheel_joint" type="continuous">
     <origin xyz="0 0 0" rpy="1.5708 0 0" />
-    <parent link="$(arg robot_name)_right_steering_hinge" />
-    <child link="$(arg robot_name)_right_front_wheel" />
+    <parent link="right_steering_hinge" />
+    <child link="right_front_wheel" />
     <axis xyz="0 0 -1" />
     <limit effort="10" velocity="100"/>
   </joint>
   <!-- Add Hokuyo laser scanner -->
-  <link name="$(arg robot_name)_laser">
+  <link name="laser">
     <inertial>
       <xacro:hokuyo_inertial_params />
@@ -266,19 +266,13 @@
     </visual>
   </link>
-  <joint name="$(arg robot_name)_hokuyo_joint" type="fixed">
+  <joint name="hokuyo_joint" type="fixed">
 	  <origin xyz="0.355 0.0 0.08" rpy="0 0 0"/>
-          <parent link="$(arg robot_name)_chassis" />
-          <child link="$(arg robot_name)_laser" />
+          <parent link="chassis" />
+          <child link="laser" />
           <axis xyz="0 0 1" />
   </joint>
   <!-- ADD ZED camera and its components -->
 <!-- base_link -->
-  <joint name="$(arg robot_name)_chassis_to_zed" type="fixed">
-	  <origin xyz="0.400 0.0 0.065" rpy="0 0 0" />
-	  <parent link="$(arg robot_name)_chassis" />
-          <child link="$(arg base_frame)" />
-	  <axis xyz="0 0 1" />
-  </joint>
-  <link name="$(arg base_frame)" />
+  <!-- <link name="$(arg base_frame)" />  -->
   <!-- Camera Center -->
     <joint name="$(arg camera_name)_camera_center_joint" type="fixed">
